Commit message: - some urdf geometry update - initial world building in gazebo

File: src/my_robot_description/urdf/cubic_doggo_legB.xacro (robot description, xacro)
@@ -273,5 +273,5 @@
         <visual>
             <geometry>
-                <sphere radius="0.013"/>
+                <sphere radius="0.008"/>
             </geometry>
             <origin xyz="0 0 0" rpy="0 0 0"/>
@@ -280,9 +280,9 @@
         <collision>
             <geometry>
-                <sphere radius="0.011"/>
+                <sphere radius="0.008"/>
             </geometry>
             <origin xyz="0 0 0" rpy="0 0 0"/>
         </collision>
-        <xacro:sphere_inertia m="0.0080" r="0.011" o_xyz="0 0 0" o_rpy="0 0 0"/>
+        <xacro:sphere_inertia m="0.004" r="0.008" o_xyz="0 0 0" o_rpy="0 0 0"/>
     </link>
     <joint name="calfFeet_calfSphere_${prefix}" type="fixed">

File: src/my_robot_description/urdf/cubic_doggo_legF.xacro (robot description, xacro)
@@ -273,5 +273,5 @@
         <visual>
             <geometry>
-                <sphere radius="0.013"/>
+                <sphere radius="0.008"/>
             </geometry>
             <origin xyz="0 0 0" rpy="0 0 0"/>
@@ -280,9 +280,9 @@
         <collision>
             <geometry>
-                <sphere radius="0.011"/>
+                <sphere radius="0.008"/>
             </geometry>
             <origin xyz="0 0 0" rpy="0 0 0"/>
         </collision>
-        <xacro:sphere_inertia m="0.0080" r="0.011" o_xyz="0 0 0" o_rpy="0 0 0"/>
+        <xacro:sphere_inertia m="0.004" r="0.008" o_xyz="0 0 0" o_rpy="0 0 0"/>
     </link>
     <joint name="calfFeet_calfSphere_${prefix}" type="fixed">
