Commit message: - adding battery weight to gazebo model preparation

File: src/my_robot_description/urdf/cubic_doggo.gazebo.xacro (robot description, xacro)
@@ -8,5 +8,5 @@
         <visual>
             <geometry>
-                <mesh filename="package://my_robot_description/mesh/CADv2/baseTorso.stl" scale="0.001 0.001 0.001"/>
+                <mesh filename="package://my_robot_description/mesh/CADv3/baseTorso.stl" scale="0.001 0.001 0.001"/>
             </geometry>
             <origin xyz="0 0 0" rpy="0 0 0"/>
@@ -24,5 +24,5 @@
         <visual>
             <geometry>
-                <mesh filename="package://my_robot_description/mesh/CADv2/basePlate.stl" scale="0.001 0.001 0.001"/>
+                <mesh filename="package://my_robot_description/mesh/CADv3/basePlate.stl" scale="0.001 0.001 0.001"/>
             </geometry>
             <origin xyz="0 0 0" rpy="0 0 0"/>
@@ -45,5 +45,5 @@
         <visual>
             <geometry>
-                <mesh filename="package://my_robot_description/mesh/CADv2/basePlate.stl" scale="0.001 0.001 0.001"/>
+                <mesh filename="package://my_robot_description/mesh/CADv3/basePlate.stl" scale="0.001 0.001 0.001"/>
             </geometry>
             <origin xyz="0 0 0" rpy="0 0 0"/>
@@ -62,4 +62,31 @@
         <child  link="base_plate_F"/>
         <origin xyz="0 0.091 0.004" rpy="0 0 ${urdf_pi}"/>
+    </joint>
+    <link name="batteryHolder">
+        <visual>
+            <geometry>
+                <mesh filename="package://my_robot_description/mesh/CADv3/batteryHolder.stl" scale="0.001 0.001 0.001"/>
+            </geometry>
+            <origin xyz="0 0 0" rpy="0 0 0"/>
+            <material name="white"/>
+        </visual>
+        <collision>
+            <geometry>
+                <mesh filename="package://my_robot_description/mesh/collisionV3/batteryHolder.stl" scale="0.001 0.001 0.001"/>
+            </geometry>
+            <origin xyz="0 0 0" rpy="0 0 0"/>
+        </collision>
+        <inertial>
+            <origin xyz="0.0 -0.0018 0.0525" rpy="0 0 0"/>
+            <mass value="0.460"/>
+            <inertia ixx="0.0008346" ixy="0" ixz="0"
+                 iyy="0.0007990" iyz="0"
+                 izz="0.0001736"/>
+        </inertial>
+    </link>
+    <joint name="torso_batteryHolder" type="fixed">
+        <parent link="base_link"/>
+        <child  link="batteryHolder"/>
+        <origin xyz="0 0 0" rpy="${urdf_pi/2} 0 0"/>
     </joint>
     <link name="imu_board">
@@ -90,4 +117,15 @@
     <xacro:doggo_legB prefix='BR'/>
 <!-- ================================================================================================================================== -->
+    <gazebo reference="batteryHolder">
+        <collision>
+            <surface>
+                <contact>
+                    <ode>
+                        <min_depth>0.001</min_depth>   <!-- enforcing convexity -->
+                    </ode>
+                </contact>
+            </surface>
+        </collision>
+    </gazebo>
     <gazebo reference="imu_board">
         <sensor name="imu_bno055" type="imu">

File: src/my_robot_description/urdf/cubic_doggo_legB.xacro (robot description, xacro)
@@ -20,5 +20,5 @@
         <visual>
             <geometry>
-                <mesh filename="package://my_robot_description/mesh/CADv2/XL430holderBasic.stl" scale="0.001 0.001 0.001"/>
+                <mesh filename="package://my_robot_description/mesh/CADv3/XL430holderBasic.stl" scale="0.001 0.001 0.001"/>
             </geometry>
             <material name="white"/>
@@ -87,5 +87,5 @@
         <visual>
             <geometry>
-                <mesh filename="package://my_robot_description/mesh/CADv2/XL430holderBasic.stl" scale="0.001 0.001 0.001"/>
+                <mesh filename="package://my_robot_description/mesh/CADv3/XL430holderBasic.stl" scale="0.001 0.001 0.001"/>
             </geometry>
             <material name="white"/>
@@ -156,5 +156,5 @@
         <visual>
             <geometry>
-                <mesh filename="package://my_robot_description/mesh/CADv2/thighInner.stl" scale="0.001 0.001 0.001"/>
+                <mesh filename="package://my_robot_description/mesh/CADv3/thighInner.stl" scale="0.001 0.001 0.001"/>
             </geometry>
             <material name="white"/>
@@ -178,5 +178,5 @@
         <visual>
             <geometry>
-                <mesh filename="package://my_robot_description/mesh/CADv2/thighOuter.stl" scale="0.001 0.001 0.001"/>
+                <mesh filename="package://my_robot_description/mesh/CADv3/thighOuter.stl" scale="0.001 0.001 0.001"/>
             </geometry>
             <material name="white"/>
@@ -222,5 +222,5 @@
         <visual>
             <geometry>
-                <mesh filename="package://my_robot_description/mesh/CADv2/calfFeetSpring.stl" scale="0.001 0.001 0.001"/>
+                <mesh filename="package://my_robot_description/mesh/CADv3/calfFeetSpring.stl" scale="0.001 0.001 0.001"/>
             </geometry>
             <material name="white"/>
@@ -247,5 +247,5 @@
         <visual>
             <geometry>
-                <mesh filename="package://my_robot_description/mesh/CADv2/calfJoint.stl" scale="0.001 0.001 0.001"/>
+                <mesh filename="package://my_robot_description/mesh/CADv3/calfJoint.stl" scale="0.001 0.001 0.001"/>
             </geometry>
             <origin xyz="0 0 0" rpy="${-urdf_pi/2} 0 ${rflc*urdf_pi/2}"/>

File: src/my_robot_description/urdf/cubic_doggo_legF.xacro (robot description, xacro)
@@ -20,5 +20,5 @@
         <visual>
             <geometry>
-                <mesh filename="package://my_robot_description/mesh/CADv2/XL430holderBasic.stl" scale="0.001 0.001 0.001"/>
+                <mesh filename="package://my_robot_description/mesh/CADv3/XL430holderBasic.stl" scale="0.001 0.001 0.001"/>
             </geometry>
             <material name="white"/>
@@ -87,5 +87,5 @@
         <visual>
             <geometry>
-                <mesh filename="package://my_robot_description/mesh/CADv2/XL430holderBasic.stl" scale="0.001 0.001 0.001"/>
+                <mesh filename="package://my_robot_description/mesh/CADv3/XL430holderBasic.stl" scale="0.001 0.001 0.001"/>
             </geometry>
             <material name="white"/>
@@ -156,5 +156,5 @@
         <visual>
             <geometry>
-                <mesh filename="package://my_robot_description/mesh/CADv2/thighInner.stl" scale="0.001 0.001 0.001"/>
+                <mesh filename="package://my_robot_description/mesh/CADv3/thighInner.stl" scale="0.001 0.001 0.001"/>
             </geometry>
             <material name="white"/>
@@ -178,5 +178,5 @@
         <visual>
             <geometry>
-                <mesh filename="package://my_robot_description/mesh/CADv2/thighOuter.stl" scale="0.001 0.001 0.001"/>
+                <mesh filename="package://my_robot_description/mesh/CADv3/thighOuter.stl" scale="0.001 0.001 0.001"/>
             </geometry>
             <material name="white"/>
@@ -222,5 +222,5 @@
         <visual>
             <geometry>
-                <mesh filename="package://my_robot_description/mesh/CADv2/calfFeetSpring.stl" scale="0.001 0.001 0.001"/>
+                <mesh filename="package://my_robot_description/mesh/CADv3/calfFeetSpring.stl" scale="0.001 0.001 0.001"/>
             </geometry>
             <material name="white"/>
@@ -247,5 +247,5 @@
         <visual>
             <geometry>
-                <mesh filename="package://my_robot_description/mesh/CADv2/calfJoint.stl" scale="0.001 0.001 0.001"/>
+                <mesh filename="package://my_robot_description/mesh/CADv3/calfJoint.stl" scale="0.001 0.001 0.001"/>
             </geometry>
             <origin xyz="0 0 0" rpy="${urdf_pi/2} 0 ${-rflc*urdf_pi/2}"/>

Commit message: - quick change for imu direction

File: src/my_robot_description/urdf/cubic_doggo.gazebo.xacro (robot description, xacro)
@@ -109,5 +109,5 @@
         <parent link="base_link"/>
         <child  link="imu_board"/>
-        <origin xyz="0.0 0.0475 -0.002" rpy="0 0 0"/>
+        <origin xyz="0.0 0.0475 -0.002" rpy="${urdf_pi} 0 ${urdf_pi}"/>
     </joint>
 <!-- ================================================================================================================================== -->
