Commit message: - adding all the main weights on the robot - update effort to 1.4 and friction parameters on the feet

File: src/my_robot_description/urdf/cubic_doggo.gazebo.xacro (robot description, xacro)
@@ -88,5 +88,131 @@
         <parent link="base_link"/>
         <child  link="batteryHolder"/>
-        <origin xyz="0 0 0" rpy="${urdf_pi/2} 0 0"/>
+        <origin xyz="0 0.089 0.03" rpy="${-urdf_pi/2} 0 ${urdf_pi}"/>
+    </joint>
+    <link name="U2D2powerHub_front">
+        <visual>
+            <geometry>
+                <mesh filename="package://my_robot_description/mesh/external/powerHubU2D2.stl" scale="0.001 0.001 0.001"/>
+            </geometry>
+            <origin xyz="0 0 0" rpy="${-urdf_pi/2} 0 ${urdf_pi}"/>
+            <material name="grey"/>
+        </visual>
+        <collision>
+            <geometry>
+                <box size="0.048 0.056 0.004"/>
+            </geometry>
+            <origin xyz="0.0005 0 0" rpy="0 0 0"/>
+        </collision>
+        <xacro:box_inertia m="0.026" x="0.048" y="0.056" z="0.004" o_xyz="0.0005 0 0" o_rpy="0 0 0"/>
+    </link>
+    <joint name="torso_U2D2powerHub_front" type="fixed">
+        <parent link="base_link"/>
+        <child  link="U2D2powerHub_front"/>
+        <origin xyz="0 0.118 -0.002" rpy="0 0 0"/>
+    </joint>
+    <link name="U2D2powerHub_back">
+        <visual>
+            <geometry>
+                <mesh filename="package://my_robot_description/mesh/external/powerHubU2D2.stl" scale="0.001 0.001 0.001"/>
+            </geometry>
+            <origin xyz="0 0 0" rpy="${-urdf_pi/2} 0 0"/>
+            <material name="grey"/>
+        </visual>
+        <collision>
+            <geometry>
+                <box size="0.048 0.056 0.004"/>
+            </geometry>
+            <origin xyz="0.0005 0 0" rpy="0 0 0"/>
+        </collision>
+        <xacro:box_inertia m="0.016" x="0.048" y="0.056" z="0.004" o_xyz="0.0005 0 0" o_rpy="0 0 0"/>
+    </link>
+    <joint name="torso_U2D2powerHub_back" type="fixed">
+        <parent link="base_link"/>
+        <child  link="U2D2powerHub_back"/>
+        <origin xyz="0 -0.094 -0.002" rpy="0 0 0"/>
+    </joint>
+    <link name="DCDCconvertor">
+        <visual>
+            <geometry>
+                <box size="0.063 0.027 0.004"/>
+            </geometry>
+            <origin xyz="0 0 0" rpy="0 0 0"/>
+            <material name="grey"/>
+        </visual>
+        <collision>
+            <geometry>
+                <box size="0.063 0.027 0.004"/>
+            </geometry>
+            <origin xyz="0 0 0" rpy="0 0 0"/>
+        </collision>
+        <xacro:box_inertia m="0.02" x="0.063" y="0.027" z="0.004" o_xyz="0 0 0" o_rpy="0 0 0"/>
+    </link>
+    <joint name="torso_DCDCconvertor" type="fixed">
+        <parent link="base_link"/>
+        <child  link="DCDCconvertor"/>
+        <origin xyz="0 0.018 -0.004" rpy="0 0 0"/>
+    </joint>
+    <link name="raspberryPi5">
+        <visual>
+            <geometry>
+                <mesh filename="package://my_robot_description/mesh/external/raspberryPi5.stl" scale="0.001 0.001 0.001"/>
+            </geometry>
+            <origin xyz="0 0 0" rpy="${urdf_pi} 0 ${urdf_pi/2}"/>
+            <material name="grey"/>
+        </visual>
+        <collision>
+            <geometry>
+                <box size="0.056 0.085 0.008"/>
+            </geometry>
+            <origin xyz="0 0 -0.004" rpy="0 0 0"/>
+        </collision>
+        <xacro:box_inertia m="0.062" x="0.056" y="0.85" z="0.008" o_xyz="0 0 -0.004" o_rpy="0 0 0"/>
+    </link>
+    <joint name="torso_raspberryPi5" type="fixed">
+        <parent link="base_link"/>
+        <child  link="raspberryPi5"/>
+        <origin xyz="0 -0.018 -0.018" rpy="0 0 0"/>
+    </joint>
+    <link name="lidarHolder">
+        <visual>
+            <geometry>
+                <mesh filename="package://my_robot_description/mesh/CADv3/lidarHolder.stl" scale="0.001 0.001 0.001"/>
+            </geometry>
+            <origin xyz="0 0 0" rpy="${urdf_pi} 0 ${urdf_pi}"/>
+            <material name="grey"/>
+        </visual>
+        <collision>
+            <geometry>
+                <box size="0.064 0.082 0.034"/>
+            </geometry>
+            <origin xyz="0 -0.009 0.013" rpy="0 0 0"/>
+        </collision>
+        <xacro:box_inertia m="0.01" x="0.064" y="0.082" z="0.034" o_xyz="0 -0.009 0.013" o_rpy="0 0 0"/>
+    </link>
+    <joint name="torso_lidarHolder" type="fixed">
+        <parent link="base_link"/>
+        <child  link="lidarHolder"/>
+        <origin xyz="0 0.136 -0.026" rpy="0 0 0"/>
+    </joint>
+    <link name="lidar_RPLIDAR_A1">
+        <visual>
+            <geometry>
+                <cylinder radius="0.035" length="0.024"/>
+            </geometry>
+            <origin xyz="0 0 0" rpy="0 0 0"/>
+            <material name="black"/>
+        </visual>
+        <collision>
+            <geometry>
+                <box size="0.07 0.095 0.05"/>
+            </geometry>
+            <origin xyz="0 -0.012 0" rpy="0 0 0"/>
+        </collision>
+        <xacro:box_inertia m="0.16" x="0.07" y="0.095" z="0.05" o_xyz="0 -0.012 0" o_rpy="0 0 0"/>
+    </link>
+    <joint name="lidarHolder_lidar_RPLIDAR_A1" type="fixed">
+        <parent link="lidarHolder"/>
+        <child  link="lidar_RPLIDAR_A1"/>
+        <origin xyz="0 0 -0.025" rpy="0 0 0"/>
     </joint>
     <link name="imu_board">
@@ -116,4 +242,19 @@
     <xacro:doggo_legB prefix='BL'/>
     <xacro:doggo_legB prefix='BR'/>
+    <xacro:macro name="foot_friction" params="prefix">
+        <gazebo reference="calfFeet_${prefix}">
+            <mu1>0.5</mu1>              <!-- Static Friction -->
+            <mu2>0.5</mu2>              <!-- Dynamic Friction -->
+            <kp>1000000.0</kp>          <!-- Contact Stiffness -->
+            <kd>1.0</kd>                <!-- Damping -->
+            <minDepth>0.001</minDepth>  <!-- Helps contact stability -->
+            <maxVel>0.1</maxVel>        <!-- Prevents "launching" on contact -->
+            <fdir1>1 0 0</fdir1>        <!-- Direction of mu1 -->
+        </gazebo>
+    </xacro:macro>
+    <xacro:foot_friction prefix="FL"/>
+    <xacro:foot_friction prefix="FR"/>
+    <xacro:foot_friction prefix="BL"/>
+    <xacro:foot_friction prefix="BR"/>
 <!-- ================================================================================================================================== -->
     <gazebo reference="batteryHolder">

File: src/my_robot_description/urdf/cubic_doggo.urdf.xacro (robot description, xacro)
@@ -10,5 +10,5 @@
         <visual>
             <geometry>
-                <mesh filename="package://my_robot_description/mesh/CADv2/baseTorso.stl" scale="0.001 0.001 0.001"/>
+                <mesh filename="package://my_robot_description/mesh/CADv3/baseTorso.stl" scale="0.001 0.001 0.001"/>
             </geometry>
             <origin xyz="0 0 0" rpy="0 0 0"/>
@@ -31,5 +31,5 @@
         <visual>
             <geometry>
-                <mesh filename="package://my_robot_description/mesh/CADv2/basePlate.stl" scale="0.001 0.001 0.001"/>
+                <mesh filename="package://my_robot_description/mesh/CADv3/basePlate.stl" scale="0.001 0.001 0.001"/>
             </geometry>
             <origin xyz="0 0 0" rpy="0 0 0"/>
@@ -52,5 +52,5 @@
         <visual>
             <geometry>
-                <mesh filename="package://my_robot_description/mesh/CADv2/basePlate.stl" scale="0.001 0.001 0.001"/>
+                <mesh filename="package://my_robot_description/mesh/CADv3/basePlate.stl" scale="0.001 0.001 0.001"/>
             </geometry>
             <origin xyz="0 0 0" rpy="0 0 0"/>
@@ -69,4 +69,157 @@
         <child  link="base_plate_F"/>
         <origin xyz="0 0.091 0.004" rpy="0 0 ${urdf_pi}"/>
+    </joint>
+    <link name="batteryHolder">
+        <visual>
+            <geometry>
+                <mesh filename="package://my_robot_description/mesh/CADv3/batteryHolder.stl" scale="0.001 0.001 0.001"/>
+            </geometry>
+            <origin xyz="0 0 0" rpy="0 0 0"/>
+            <material name="white"/>
+        </visual>
+        <collision>
+            <geometry>
+                <mesh filename="package://my_robot_description/mesh/collisionV3/batteryHolder.stl" scale="0.001 0.001 0.001"/>
+            </geometry>
+            <origin xyz="0 0 0" rpy="0 0 0"/>
+        </collision>
+        <inertial>
+            <origin xyz="0.0 -0.0018 0.0525" rpy="0 0 0"/>
+            <mass value="0.460"/>
+            <inertia ixx="0.0008346" ixy="0" ixz="0"
+                 iyy="0.0007990" iyz="0"
+                 izz="0.0001736"/>
+        </inertial>
+    </link>
+    <joint name="torso_batteryHolder" type="fixed">
+        <parent link="base_link"/>
+        <child  link="batteryHolder"/>
+        <origin xyz="0 0.089 0.03" rpy="${-urdf_pi/2} 0 ${urdf_pi}"/>
+    </joint>
+    <link name="U2D2powerHub_front">
+        <visual>
+            <geometry>
+                <mesh filename="package://my_robot_description/mesh/external/powerHubU2D2.stl" scale="0.001 0.001 0.001"/>
+            </geometry>
+            <origin xyz="0 0 0" rpy="${-urdf_pi/2} 0 ${urdf_pi}"/>
+            <material name="grey"/>
+        </visual>
+        <collision>
+            <geometry>
+                <box size="0.048 0.056 0.004"/>
+            </geometry>
+            <origin xyz="0.0005 0 0" rpy="0 0 0"/>
+        </collision>
+        <xacro:box_inertia m="0.026" x="0.048" y="0.056" z="0.004" o_xyz="0.0005 0 0" o_rpy="0 0 0"/>
+    </link>
+    <joint name="torso_U2D2powerHub_front" type="fixed">
+        <parent link="base_link"/>
+        <child  link="U2D2powerHub_front"/>
+        <origin xyz="0 0.118 -0.002" rpy="0 0 0"/>
+    </joint>
+    <link name="U2D2powerHub_back">
+        <visual>
+            <geometry>
+                <mesh filename="package://my_robot_description/mesh/external/powerHubU2D2.stl" scale="0.001 0.001 0.001"/>
+            </geometry>
+            <origin xyz="0 0 0" rpy="${-urdf_pi/2} 0 0"/>
+            <material name="grey"/>
+        </visual>
+        <collision>
+            <geometry>
+                <box size="0.048 0.056 0.004"/>
+            </geometry>
+            <origin xyz="0.0005 0 0" rpy="0 0 0"/>
+        </collision>
+        <xacro:box_inertia m="0.016" x="0.048" y="0.056" z="0.004" o_xyz="0.0005 0 0" o_rpy="0 0 0"/>
+    </link>
+    <joint name="torso_U2D2powerHub_back" type="fixed">
+        <parent link="base_link"/>
+        <child  link="U2D2powerHub_back"/>
+        <origin xyz="0 -0.094 -0.002" rpy="0 0 0"/>
+    </joint>
+    <link name="DCDCconvertor">
+        <visual>
+            <geometry>
+                <box size="0.063 0.027 0.004"/>
+            </geometry>
+            <origin xyz="0 0 0" rpy="0 0 0"/>
+            <material name="grey"/>
+        </visual>
+        <collision>
+            <geometry>
+                <box size="0.063 0.027 0.004"/>
+            </geometry>
+            <origin xyz="0 0 0" rpy="0 0 0"/>
+        </collision>
+        <xacro:box_inertia m="0.02" x="0.063" y="0.027" z="0.004" o_xyz="0 0 0" o_rpy="0 0 0"/>
+    </link>
+    <joint name="torso_DCDCconvertor" type="fixed">
+        <parent link="base_link"/>
+        <child  link="DCDCconvertor"/>
+        <origin xyz="0 0.018 -0.004" rpy="0 0 0"/>
+    </joint>
+    <link name="raspberryPi5">
+        <visual>
+            <geometry>
+                <mesh filename="package://my_robot_description/mesh/external/raspberryPi5.stl" scale="0.001 0.001 0.001"/>
+            </geometry>
+            <origin xyz="0 0 0" rpy="${urdf_pi} 0 ${urdf_pi/2}"/>
+            <material name="grey"/>
+        </visual>
+        <collision>
+            <geometry>
+                <box size="0.056 0.085 0.008"/>
+            </geometry>
+            <origin xyz="0 0 -0.004" rpy="0 0 0"/>
+        </collision>
+        <xacro:box_inertia m="0.062" x="0.056" y="0.85" z="0.008" o_xyz="0 0 -0.004" o_rpy="0 0 0"/>
+    </link>
+    <joint name="torso_raspberryPi5" type="fixed">
+        <parent link="base_link"/>
+        <child  link="raspberryPi5"/>
+        <origin xyz="0 -0.018 -0.018" rpy="0 0 0"/>
+    </joint>
+    <link name="lidarHolder">
+        <visual>
+            <geometry>
+                <mesh filename="package://my_robot_description/mesh/CADv3/lidarHolder.stl" scale="0.001 0.001 0.001"/>
+            </geometry>
+            <origin xyz="0 0 0" rpy="${urdf_pi} 0 ${urdf_pi}"/>
+            <material name="grey"/>
+        </visual>
+        <collision>
+            <geometry>
+                <box size="0.064 0.082 0.034"/>
+            </geometry>
+            <origin xyz="0 -0.009 0.013" rpy="0 0 0"/>
+        </collision>
+        <xacro:box_inertia m="0.01" x="0.064" y="0.082" z="0.034" o_xyz="0 -0.009 0.013" o_rpy="0 0 0"/>
+    </link>
+    <joint name="torso_lidarHolder" type="fixed">
+        <parent link="base_link"/>
+        <child  link="lidarHolder"/>
+        <origin xyz="0 0.136 -0.026" rpy="0 0 0"/>
+    </joint>
+    <link name="lidar_RPLIDAR_A1">
+        <visual>
+            <geometry>
+                <cylinder radius="0.035" length="0.024"/>
+            </geometry>
+            <origin xyz="0 0 0" rpy="0 0 0"/>
+            <material name="black"/>
+        </visual>
+        <collision>
+            <geometry>
+                <box size="0.07 0.095 0.05"/>
+            </geometry>
+            <origin xyz="0 -0.012 0" rpy="0 0 0"/>
+        </collision>
+        <xacro:box_inertia m="0.16" x="0.07" y="0.095" z="0.05" o_xyz="0 -0.012 0" o_rpy="0 0 0"/>
+    </link>
+    <joint name="lidarHolder_lidar_RPLIDAR_A1" type="fixed">
+        <parent link="lidarHolder"/>
+        <child  link="lidar_RPLIDAR_A1"/>
+        <origin xyz="0 0 -0.025" rpy="0 0 0"/>
     </joint>
 <!-- ================================================================================================================================== -->

File: src/my_robot_description/urdf/cubic_doggo_legB.xacro (robot description, xacro)
@@ -80,6 +80,6 @@
         <origin xyz="0 ${-servo_z/2-0.002} ${0.01+0.0025/2}" rpy="0 0 0"/>
         <axis xyz="0 -1 0"/>
-        <limit effort="1000.0" velocity="50.0" lower="${urdf_pi - urdf_pi/3}" upper="${urdf_pi + urdf_pi/3}"/>
-        <dynamics friction="0.05" damping="0.1"/>
+        <limit effort="1.4" velocity="10.0" lower="${urdf_pi - urdf_pi/3}" upper="${urdf_pi + urdf_pi/3}"/>
+        <dynamics friction="0.01" damping="0.1"/>
     </joint>
     <!-- ============================================================================================================================== -->
@@ -148,7 +148,7 @@
         <origin xyz="${rflc*(servo_z/2+0.002)} -0.01125 0" rpy="0 0 0"/>
         <axis xyz="${rflc} 0 0"/>
-        <limit effort="1000.0" velocity="50.0" lower="${urdf_pi - 2*urdf_pi/6 + rflc*urdf_pi/6}"
-                                               upper="${urdf_pi + 2*urdf_pi/6 + rflc*urdf_pi/6}"/>
-        <dynamics friction="0.05" damping="0.1"/>
+        <limit effort="1.4" velocity="10.0" lower="${urdf_pi - 2*urdf_pi/6 + rflc*urdf_pi/6}"
+                                            upper="${urdf_pi + 2*urdf_pi/6 + rflc*urdf_pi/6}"/>
+        <dynamics friction="0.01" damping="0.1"/>
     </joint>
     <!-- ============================================================================================================================== -->
@@ -241,6 +241,6 @@
         <origin xyz="${rflc*(-servo_z/2-0.002-0.0025)} ${-0.086+0.004} 0" rpy="${urdf_pi} 0 0"/>
         <axis xyz="${-rflc} 0 0"/>
-        <limit effort="1000.0" velocity="50.0" lower="${5*urdf_pi/8}" upper="${11*urdf_pi/8}"/>
-        <dynamics friction="0.0128" damping="0.1"/>
+        <limit effort="1.4" velocity="10.0" lower="${5*urdf_pi/8}" upper="${11*urdf_pi/8}"/>
+        <dynamics friction="0.01" damping="0.1"/>
     </joint>
     <link name="calfJoint_${prefix}">
@@ -267,6 +267,6 @@
         <axis xyz="${-rflc} 0 0"/>
         <mimic joint="servo3_calfFeet_${prefix}" multiplier="1.0" offset="0.0"/>
-        <limit effort="1000.0" velocity="50.0" lower="${5*urdf_pi/8}" upper="${11*urdf_pi/8}"/>
-        <dynamics friction="0.0212" damping="0.1"/>
+        <limit effort="1.4" velocity="10.0" lower="${5*urdf_pi/8}" upper="${11*urdf_pi/8}"/>
+        <dynamics friction="0.01" damping="0.1"/>
     </joint>
     <link name="calfSphere_${prefix}">

File: src/my_robot_description/urdf/cubic_doggo_legF.xacro (robot description, xacro)
@@ -80,6 +80,6 @@
         <origin xyz="0 ${-servo_z/2-0.002} ${0.01+0.0025/2}" rpy="0 0 0"/>
         <axis xyz="0 -1 0"/>
-        <limit effort="1000.0" velocity="50.0" lower="${urdf_pi - urdf_pi/3}" upper="${urdf_pi + urdf_pi/3}"/>
-        <dynamics friction="0.05" damping="0.1"/>
+        <limit effort="1.4" velocity="10.0" lower="${urdf_pi - urdf_pi/3}" upper="${urdf_pi + urdf_pi/3}"/>
+        <dynamics friction="0.01" damping="0.1"/>
     </joint>
     <!-- ============================================================================================================================== -->
@@ -148,7 +148,7 @@
         <origin xyz="${rflc*(servo_z/2+0.002)} -0.03525 0" rpy="0 0 0"/>
         <axis xyz="${rflc} 0 0"/>
-        <limit effort="1000.0" velocity="50.0" lower="${urdf_pi - 2*urdf_pi/6 - rflc*urdf_pi/6}"
+        <limit effort="1.4" velocity="10.0" lower="${urdf_pi - 2*urdf_pi/6 - rflc*urdf_pi/6}"
                                                upper="${urdf_pi + 2*urdf_pi/6 - rflc*urdf_pi/6}"/>
-        <dynamics friction="0.05" damping="0.1"/>
+        <dynamics friction="0.01" damping="0.1"/>
     </joint>
     <!-- ============================================================================================================================== -->
@@ -241,6 +241,6 @@
         <origin xyz="${rflc*(-servo_z/2-0.002-0.0025)} ${-0.086+0.004} 0" rpy="0 0 0"/>
         <axis xyz="${-rflc} 0 0"/>
-        <limit effort="1000.0" velocity="50.0" lower="${5*urdf_pi/8}" upper="${11*urdf_pi/8}"/>
-        <dynamics friction="0.0128" damping="0.1"/>
+        <limit effort="1.4" velocity="10.0" lower="${5*urdf_pi/8}" upper="${11*urdf_pi/8}"/>
+        <dynamics friction="0.01" damping="0.1"/>
     </joint>
     <link name="calfJoint_${prefix}">
@@ -267,6 +267,6 @@
         <axis xyz="${-rflc} 0 0"/>
         <mimic joint="servo3_calfFeet_${prefix}" multiplier="1.0" offset="0.0"/>
-        <limit effort="1000.0" velocity="50.0" lower="${5*urdf_pi/8}" upper="${11*urdf_pi/8}"/>
-        <dynamics friction="0.0212" damping="0.1"/>
+        <limit effort="1.4" velocity="10.0" lower="${5*urdf_pi/8}" upper="${11*urdf_pi/8}"/>
+        <dynamics friction="0.01" damping="0.1"/>
     </joint>
     <link name="calfSphere_${prefix}">

Commit message: - some patching up for the Gazebo simulation

File: src/my_robot_description/urdf/cubic_doggo.gazebo.xacro (robot description, xacro)
@@ -207,5 +207,5 @@
                 <box size="0.07 0.095 0.05"/>
             </geometry>
-            <origin xyz="0 -0.012 0" rpy="0 0 0"/>
+            <origin xyz="0 -0.012 0.012" rpy="0 0 0"/>
         </collision>
         <xacro:box_inertia m="0.16" x="0.07" y="0.095" z="0.05" o_xyz="0 -0.012 0" o_rpy="0 0 0"/>
@@ -214,5 +214,5 @@
         <parent link="lidarHolder"/>
         <child  link="lidar_RPLIDAR_A1"/>
-        <origin xyz="0 0 -0.025" rpy="0 0 0"/>
+        <origin xyz="0 0 -0.041" rpy="0 0 0"/>
     </joint>
     <link name="imu_board">

File: src/my_robot_description/urdf/cubic_doggo.urdf.xacro (robot description, xacro)
@@ -214,5 +214,5 @@
                 <box size="0.07 0.095 0.05"/>
             </geometry>
-            <origin xyz="0 -0.012 0" rpy="0 0 0"/>
+            <origin xyz="0 -0.012 0.012" rpy="0 0 0"/>
         </collision>
         <xacro:box_inertia m="0.16" x="0.07" y="0.095" z="0.05" o_xyz="0 -0.012 0" o_rpy="0 0 0"/>
@@ -221,5 +221,5 @@
         <parent link="lidarHolder"/>
         <child  link="lidar_RPLIDAR_A1"/>
-        <origin xyz="0 0 -0.025" rpy="0 0 0"/>
+        <origin xyz="0 0 -0.041" rpy="0 0 0"/>
     </joint>
 <!-- ================================================================================================================================== -->

File: src/my_robot_description/urdf/cubic_doggo_legB.xacro (robot description, xacro)
@@ -289,5 +289,5 @@
         <parent link="calfFeet_${prefix}"/>
         <child  link="calfSphere_${prefix}"/>
-        <origin xyz="0 -0.004 ${-0.105+0.035}" rpy="0 0 0"/>
+        <origin xyz="0 -0.002 ${-0.105+0.035}" rpy="0 0 0"/>
     </joint>
     </xacro:macro>

File: src/my_robot_description/urdf/cubic_doggo_legF.xacro (robot description, xacro)
@@ -289,5 +289,5 @@
         <parent link="calfFeet_${prefix}"/>
         <child  link="calfSphere_${prefix}"/>
-        <origin xyz="0 0.004 ${-0.105+0.035}" rpy="0 0 0"/>
+        <origin xyz="0 0.002 ${-0.105+0.035}" rpy="0 0 0"/>
     </joint>
     </xacro:macro>
