Commit message: - separate out the load to its own cubic_doggo_load.xacro, so that it's not repeated sim vs real

File: src/my_robot_description/urdf/cubic_doggo.gazebo.xacro (robot description, xacro)
@@ -4,4 +4,5 @@
     <xacro:include filename="cubic_doggo_legF.xacro"/>
     <xacro:include filename="cubic_doggo_legB.xacro"/>
+    <xacro:include filename="cubic_doggo_load.xacro"/>
 <!-- ================================================================================================================================== -->
     <link name="base_link">
@@ -62,157 +63,4 @@
         <child  link="base_plate_F"/>
         <origin xyz="0 0.091 0.004" rpy="0 0 ${urdf_pi}"/>
-    </joint>
-    <link name="batteryHolder">
-        <visual>
-            <geometry>
-                <mesh filename="package://my_robot_description/mesh/CADv3/batteryHolder.stl" scale="0.001 0.001 0.001"/>
-            </geometry>
-            <origin xyz="0 0 0" rpy="0 0 0"/>
-            <material name="white"/>
-        </visual>
-        <collision>
-            <geometry>
-                <mesh filename="package://my_robot_description/mesh/collisionV3/batteryHolder.stl" scale="0.001 0.001 0.001"/>
-            </geometry>
-            <origin xyz="0 0 0" rpy="0 0 0"/>
-        </collision>
-        <inertial>
-            <origin xyz="0.0 -0.0018 0.0525" rpy="0 0 0"/>
-            <mass value="0.460"/>
-            <inertia ixx="0.0008346" ixy="0" ixz="0"
-                 iyy="0.0007990" iyz="0"
-                 izz="0.0001736"/>
-        </inertial>
-    </link>
-    <joint name="torso_batteryHolder" type="fixed">
-        <parent link="base_link"/>
-        <child  link="batteryHolder"/>
-        <origin xyz="0 0.089 0.03" rpy="${-urdf_pi/2} 0 ${urdf_pi}"/>
-    </joint>
-    <link name="U2D2powerHub_front">
-        <visual>
-            <geometry>
-                <mesh filename="package://my_robot_description/mesh/external/powerHubU2D2.stl" scale="0.001 0.001 0.001"/>
-            </geometry>
-            <origin xyz="0 0 0" rpy="${-urdf_pi/2} 0 ${urdf_pi}"/>
-            <material name="grey"/>
-        </visual>
-        <collision>
-            <geometry>
-                <box size="0.048 0.056 0.004"/>
-            </geometry>
-            <origin xyz="0.0005 0 0" rpy="0 0 0"/>
-        </collision>
-        <xacro:box_inertia m="0.026" x="0.048" y="0.056" z="0.004" o_xyz="0.0005 0 0" o_rpy="0 0 0"/>
-    </link>
-    <joint name="torso_U2D2powerHub_front" type="fixed">
-        <parent link="base_link"/>
-        <child  link="U2D2powerHub_front"/>
-        <origin xyz="0 0.118 -0.002" rpy="0 0 0"/>
-    </joint>
-    <link name="U2D2powerHub_back">
-        <visual>
-            <geometry>
-                <mesh filename="package://my_robot_description/mesh/external/powerHubU2D2.stl" scale="0.001 0.001 0.001"/>
-            </geometry>
-            <origin xyz="0 0 0" rpy="${-urdf_pi/2} 0 0"/>
-            <material name="grey"/>
-        </visual>
-        <collision>
-            <geometry>
-                <box size="0.048 0.056 0.004"/>
-            </geometry>
-            <origin xyz="0.0005 0 0" rpy="0 0 0"/>
-        </collision>
-        <xacro:box_inertia m="0.016" x="0.048" y="0.056" z="0.004" o_xyz="0.0005 0 0" o_rpy="0 0 0"/>
-    </link>
-    <joint name="torso_U2D2powerHub_back" type="fixed">
-        <parent link="base_link"/>
-        <child  link="U2D2powerHub_back"/>
-        <origin xyz="0 -0.094 -0.002" rpy="0 0 0"/>
-    </joint>
-    <link name="DCDCconvertor">
-        <visual>
-            <geometry>
-                <box size="0.063 0.027 0.004"/>
-            </geometry>
-            <origin xyz="0 0 0" rpy="0 0 0"/>
-            <material name="grey"/>
-        </visual>
-        <collision>
-            <geometry>
-                <box size="0.063 0.027 0.004"/>
-            </geometry>
-            <origin xyz="0 0 0" rpy="0 0 0"/>
-        </collision>
-        <xacro:box_inertia m="0.02" x="0.063" y="0.027" z="0.004" o_xyz="0 0 0" o_rpy="0 0 0"/>
-    </link>
-    <joint name="torso_DCDCconvertor" type="fixed">
-        <parent link="base_link"/>
-        <child  link="DCDCconvertor"/>
-        <origin xyz="0 0.018 -0.004" rpy="0 0 0"/>
-    </joint>
-    <link name="raspberryPi5">
-        <visual>
-            <geometry>
-                <mesh filename="package://my_robot_description/mesh/external/raspberryPi5.stl" scale="0.001 0.001 0.001"/>
-            </geometry>
-            <origin xyz="0 0 0" rpy="${urdf_pi} 0 ${urdf_pi/2}"/>
-            <material name="grey"/>
-        </visual>
-        <collision>
-            <geometry>
-                <box size="0.056 0.085 0.008"/>
-            </geometry>
-            <origin xyz="0 0 -0.004" rpy="0 0 0"/>
-        </collision>
-        <xacro:box_inertia m="0.062" x="0.056" y="0.85" z="0.008" o_xyz="0 0 -0.004" o_rpy="0 0 0"/>
-    </link>
-    <joint name="torso_raspberryPi5" type="fixed">
-        <parent link="base_link"/>
-        <child  link="raspberryPi5"/>
-        <origin xyz="0 -0.018 -0.018" rpy="0 0 0"/>
-    </joint>
-    <link name="lidarHolder">
-        <visual>
-            <geometry>
-                <mesh filename="package://my_robot_description/mesh/CADv3/lidarHolder.stl" scale="0.001 0.001 0.001"/>
-            </geometry>
-            <origin xyz="0 0 0" rpy="${urdf_pi} 0 ${urdf_pi}"/>
-            <material name="grey"/>
-        </visual>
-        <collision>
-            <geometry>
-                <box size="0.064 0.082 0.034"/>
-            </geometry>
-            <origin xyz="0 -0.009 0.013" rpy="0 0 0"/>
-        </collision>
-        <xacro:box_inertia m="0.01" x="0.064" y="0.082" z="0.034" o_xyz="0 -0.009 0.013" o_rpy="0 0 0"/>
-    </link>
-    <joint name="torso_lidarHolder" type="fixed">
-        <parent link="base_link"/>
-        <child  link="lidarHolder"/>
-        <origin xyz="0 0.136 -0.026" rpy="0 0 0"/>
-    </joint>
-    <link name="lidar_RPLIDAR_A1">
-        <visual>
-            <geometry>
-                <cylinder radius="0.035" length="0.024"/>
-            </geometry>
-            <origin xyz="0 0 0" rpy="0 0 0"/>
-            <material name="black"/>
-        </visual>
-        <collision>
-            <geometry>
-                <box size="0.07 0.095 0.05"/>
-            </geometry>
-            <origin xyz="0 -0.012 0.012" rpy="0 0 0"/>
-        </collision>
-        <xacro:box_inertia m="0.16" x="0.07" y="0.095" z="0.05" o_xyz="0 -0.012 0" o_rpy="0 0 0"/>
-    </link>
-    <joint name="lidarHolder_lidar_RPLIDAR_A1" type="fixed">
-        <parent link="lidarHolder"/>
-        <child  link="lidar_RPLIDAR_A1"/>
-        <origin xyz="0 0 -0.041" rpy="0 0 0"/>
     </joint>
     <link name="imu_board">
@@ -242,4 +90,5 @@
     <xacro:doggo_legB prefix='BL'/>
     <xacro:doggo_legB prefix='BR'/>
+    <xacro:doggo_load/>
     <xacro:macro name="foot_friction" params="prefix">
         <gazebo reference="calfFeet_${prefix}">

File: src/my_robot_description/urdf/cubic_doggo.urdf.xacro (robot description, xacro)
@@ -4,4 +4,5 @@
     <xacro:include filename="cubic_doggo_legF.xacro"/>
     <xacro:include filename="cubic_doggo_legB.xacro"/>
+    <xacro:include filename="cubic_doggo_load.xacro"/>
     <xacro:include filename="cubic_doggo.ros2_control.xacro"/>
 <!-- ================================================================================================================================== -->
@@ -70,157 +71,4 @@
         <origin xyz="0 0.091 0.004" rpy="0 0 ${urdf_pi}"/>
     </joint>
-    <link name="batteryHolder">
-        <visual>
-            <geometry>
-                <mesh filename="package://my_robot_description/mesh/CADv3/batteryHolder.stl" scale="0.001 0.001 0.001"/>
-            </geometry>
-            <origin xyz="0 0 0" rpy="0 0 0"/>
-            <material name="white"/>
-        </visual>
-        <collision>
-            <geometry>
-                <mesh filename="package://my_robot_description/mesh/collisionV3/batteryHolder.stl" scale="0.001 0.001 0.001"/>
-            </geometry>
-            <origin xyz="0 0 0" rpy="0 0 0"/>
-        </collision>
-        <inertial>
-            <origin xyz="0.0 -0.0018 0.0525" rpy="0 0 0"/>
-            <mass value="0.460"/>
-            <inertia ixx="0.0008346" ixy="0" ixz="0"
-                 iyy="0.0007990" iyz="0"
-                 izz="0.0001736"/>
-        </inertial>
-    </link>
-    <joint name="torso_batteryHolder" type="fixed">
-        <parent link="base_link"/>
-        <child  link="batteryHolder"/>
-        <origin xyz="0 0.089 0.03" rpy="${-urdf_pi/2} 0 ${urdf_pi}"/>
-    </joint>
-    <link name="U2D2powerHub_front">
-        <visual>
-            <geometry>
-                <mesh filename="package://my_robot_description/mesh/external/powerHubU2D2.stl" scale="0.001 0.001 0.001"/>
-            </geometry>
-            <origin xyz="0 0 0" rpy="${-urdf_pi/2} 0 ${urdf_pi}"/>
-            <material name="grey"/>
-        </visual>
-        <collision>
-            <geometry>
-                <box size="0.048 0.056 0.004"/>
-            </geometry>
-            <origin xyz="0.0005 0 0" rpy="0 0 0"/>
-        </collision>
-        <xacro:box_inertia m="0.026" x="0.048" y="0.056" z="0.004" o_xyz="0.0005 0 0" o_rpy="0 0 0"/>
-    </link>
-    <joint name="torso_U2D2powerHub_front" type="fixed">
-        <parent link="base_link"/>
-        <child  link="U2D2powerHub_front"/>
-        <origin xyz="0 0.118 -0.002" rpy="0 0 0"/>
-    </joint>
-    <link name="U2D2powerHub_back">
-        <visual>
-            <geometry>
-                <mesh filename="package://my_robot_description/mesh/external/powerHubU2D2.stl" scale="0.001 0.001 0.001"/>
-            </geometry>
-            <origin xyz="0 0 0" rpy="${-urdf_pi/2} 0 0"/>
-            <material name="grey"/>
-        </visual>
-        <collision>
-            <geometry>
-                <box size="0.048 0.056 0.004"/>
-            </geometry>
-            <origin xyz="0.0005 0 0" rpy="0 0 0"/>
-        </collision>
-        <xacro:box_inertia m="0.016" x="0.048" y="0.056" z="0.004" o_xyz="0.0005 0 0" o_rpy="0 0 0"/>
-    </link>
-    <joint name="torso_U2D2powerHub_back" type="fixed">
-        <parent link="base_link"/>
-        <child  link="U2D2powerHub_back"/>
-        <origin xyz="0 -0.094 -0.002" rpy="0 0 0"/>
-    </joint>
-    <link name="DCDCconvertor">
-        <visual>
-            <geometry>
-                <box size="0.063 0.027 0.004"/>
-            </geometry>
-            <origin xyz="0 0 0" rpy="0 0 0"/>
-            <material name="grey"/>
-        </visual>
-        <collision>
-            <geometry>
-                <box size="0.063 0.027 0.004"/>
-            </geometry>
-            <origin xyz="0 0 0" rpy="0 0 0"/>
-        </collision>
-        <xacro:box_inertia m="0.02" x="0.063" y="0.027" z="0.004" o_xyz="0 0 0" o_rpy="0 0 0"/>
-    </link>
-    <joint name="torso_DCDCconvertor" type="fixed">
-        <parent link="base_link"/>
-        <child  link="DCDCconvertor"/>
-        <origin xyz="0 0.018 -0.004" rpy="0 0 0"/>
-    </joint>
-    <link name="raspberryPi5">
-        <visual>
-            <geometry>
-                <mesh filename="package://my_robot_description/mesh/external/raspberryPi5.stl" scale="0.001 0.001 0.001"/>
-            </geometry>
-            <origin xyz="0 0 0" rpy="${urdf_pi} 0 ${urdf_pi/2}"/>
-            <material name="grey"/>
-        </visual>
-        <collision>
-            <geometry>
-                <box size="0.056 0.085 0.008"/>
-            </geometry>
-            <origin xyz="0 0 -0.004" rpy="0 0 0"/>
-        </collision>
-        <xacro:box_inertia m="0.062" x="0.056" y="0.85" z="0.008" o_xyz="0 0 -0.004" o_rpy="0 0 0"/>
-    </link>
-    <joint name="torso_raspberryPi5" type="fixed">
-        <parent link="base_link"/>
-        <child  link="raspberryPi5"/>
-        <origin xyz="0 -0.018 -0.018" rpy="0 0 0"/>
-    </joint>
-    <link name="lidarHolder">
-        <visual>
-            <geometry>
-                <mesh filename="package://my_robot_description/mesh/CADv3/lidarHolder.stl" scale="0.001 0.001 0.001"/>
-            </geometry>
-            <origin xyz="0 0 0" rpy="${urdf_pi} 0 ${urdf_pi}"/>
-            <material name="grey"/>
-        </visual>
-        <collision>
-            <geometry>
-                <box size="0.064 0.082 0.034"/>
-            </geometry>
-            <origin xyz="0 -0.009 0.013" rpy="0 0 0"/>
-        </collision>
-        <xacro:box_inertia m="0.01" x="0.064" y="0.082" z="0.034" o_xyz="0 -0.009 0.013" o_rpy="0 0 0"/>
-    </link>
-    <joint name="torso_lidarHolder" type="fixed">
-        <parent link="base_link"/>
-        <child  link="lidarHolder"/>
-        <origin xyz="0 0.136 -0.026" rpy="0 0 0"/>
-    </joint>
-    <link name="lidar_RPLIDAR_A1">
-        <visual>
-            <geometry>
-                <cylinder radius="0.035" length="0.024"/>
-            </geometry>
-            <origin xyz="0 0 0" rpy="0 0 0"/>
-            <material name="black"/>
-        </visual>
-        <collision>
-            <geometry>
-                <box size="0.07 0.095 0.05"/>
-            </geometry>
-            <origin xyz="0 -0.012 0.012" rpy="0 0 0"/>
-        </collision>
-        <xacro:box_inertia m="0.16" x="0.07" y="0.095" z="0.05" o_xyz="0 -0.012 0" o_rpy="0 0 0"/>
-    </link>
-    <joint name="lidarHolder_lidar_RPLIDAR_A1" type="fixed">
-        <parent link="lidarHolder"/>
-        <child  link="lidar_RPLIDAR_A1"/>
-        <origin xyz="0 0 -0.041" rpy="0 0 0"/>
-    </joint>
 <!-- ================================================================================================================================== -->
     <xacro:doggo_legF prefix='FL'/>
@@ -228,4 +76,5 @@
     <xacro:doggo_legB prefix='BL'/>
     <xacro:doggo_legB prefix='BR'/>
+    <xacro:doggo_load/>
 <!-- ================================================================================================================================== -->
 </robot>
