Commit message: - 1 leg in mujoco configured

File: src/my_robot_description/urdf/cubic_legF.xacro (robot description, xacro)
@@ -105,5 +105,5 @@
         <origin xyz="0 -0.004 0" rpy="0 0 0"/>
     </joint>
-    <!--link name="servo2_${prefix}">
+    <link name="servo2_${prefix}">
         <visual>
             <geometry>
@@ -149,9 +149,9 @@
         <axis xyz="${rflc} 0 0"/>
         <limit effort="1.4" velocity="10.0" lower="${urdf_pi - 2*urdf_pi/6 - rflc*urdf_pi/6}"
-                                               upper="${urdf_pi + 2*urdf_pi/6 - rflc*urdf_pi/6}"/>
-        <dynamics friction="0.01" damping="0.1"/>
-    </joint-->
+                                            upper="${urdf_pi + 2*urdf_pi/6 - rflc*urdf_pi/6}"/>
+        <dynamics friction="0.01" damping="0.1"/>
+    </joint>
     <!-- ============================================================================================================================== -->
-    <!--link name="inner_thigh_${prefix}">
+    <link name="inner_thigh_${prefix}">
         <visual>
             <geometry>
@@ -290,5 +290,5 @@
         <child  link="calfSphere_${prefix}"/>
         <origin xyz="0 0.002 ${-0.105+0.035}" rpy="0 0 0"/>
-    </joint-->
+    </joint>
     </xacro:macro>
 </robot>
